File: board/rainbow-led.kicad_sch (KiCad schematic)
At the start: 9 parts, among them J1 Conn_01x04, J2 Conn_01x06, J3 Conn_01x02, SW1 SW_Push, U1 TPS61222DCKR, U3 ATtiny85-20S

Commit message: Switch inductor to recommended one.
Parts:
- removed L2: 4.7u, LQM2HPN4R7MG0L:INDC2520X100N, symbol Digikey_LQM2HPN4R7MG0L:LQM2HPN4R7MG0L
- added L1: LQH3NPN4R7MMEL, LQH3NPN4R7MMELCT:IND_LQH3NPN4R7MMEL, symbol Digikey_LQH3NPN4R7MMELCT:LQH3NPN4R7MMEL
Connections:
- net +BATT: now also L1.2
- net at U1.5 (L): now also L1.1
Changed lines of the file:
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@@
 	(wire
 		(pts
-			(xy 50.8 77.47) (xy 55.88 77.47)
+			(xy 55.88 85.09) (xy 55.88 87.63)
 		)
 		(stroke
@@
 	(wire
 		(pts
-			(xy 21.59 91.44) (xy 31.75 91.44)
+			(xy 50.8 87.63) (xy 55.88 87.63)
 		)
 		(stroke
@@
 	(wire
 		(pts
-			(xy 55.88 77.47) (xy 55.88 74.93)
+			(xy 21.59 91.44) (xy 31.75 91.44)
 		)
 		(stroke
@@
 	(wire
 		(pts
-			(xy 50.8 54.61) (xy 50.8 77.47)
+			(xy 50.8 54.61) (xy 50.8 87.63)
 		)
 		(stroke
@@
 	)
 	(symbol
+		(lib_id "Digikey_LQH3NPN4R7MMELCT:LQH3NPN4R7MMEL")
+		(at 55.88 72.39 270)
+		(unit 1)
+		(exclude_from_sim no)
+		(in_bom yes)
+		(on_board yes)
+		(dnp no)
+		(fields_autoplaced yes)
+		(property "Reference" "L1"
+			(at 58.42 71.1199 90)
+			(effects
+				(font
+					(size 1.27 1.27)
+				)
+				(justify left)
+			)
+		)
+		(property "Value" "LQH3NPN4R7MMEL"
+			(at 58.42 73.6599 90)
+			(effects
+				(font
+					(size 1.27 1.27)
+				)
+				(justify left)
+			)
+		)
+		(property "Footprint" "LQH3NPN4R7MMELCT:IND_LQH3NPN4R7MMEL"
+			(at 55.88 72.39 0)
+			(effects
+				(font
+					(size 1.27 1.27)
+				)
+				(justify bottom)
+				(hide yes)
+			)
+		)
+		(property "Datasheet" ""
+			(at 55.88 72.39 0)
+			(effects
+				(font
+					(size 1.27 1.27)
+				)
+				(hide yes)
+			)
+		)
+		(property "Description" ""
+			(at 55.88 72.39 0)
+			(effects
+				(font
+					(size 1.27 1.27)
+				)
+				(hide yes)
+			)
+		)
+		(property "PARTREV" "N/A"
+			(at 55.88 72.39 0)
+			(effects
+				(font
+					(size 1.27 1.27)
+				)
+				(justify bottom)
+				(hide yes)
+			)
+		)
+		(property "MANUFACTURER" "Murata"
+			(at 55.88 72.39 0)
+			(effects
+				(font
+					(size 1.27 1.27)
+				)
+				(justify bottom)
+				(hide yes)
+			)
+		)
+		(property "MAXIMUM_PACKAGE_HEIGHT" "1.5mm"
+			(at 55.88 72.39 0)
+			(effects
+				(font
+					(size 1.27 1.27)
+				)
+				(justify bottom)
+				(hide yes)
+			)
+		)
+		(property "STANDARD" "Manufacturer Recommendations"
+			(at 55.88 72.39 0)
+			(effects
+				(font
+					(size 1.27 1.27)
+				)
+				(justify bottom)
+				(hide yes)
+			)
+		)
+		(pin "2"
+		)
+		(pin "1"
+		)
+		(instances
+			(project ""
+				(path "/4a165a6f-6392-4b15-974f-3ac6900bac37"
+					(reference "L1")
+					(unit 1)
+				)
+			)
+		)
+	)
+	(symbol
 		(lib_id "Device:C_Small")
 		(at 101.6 54.61 180)
@@
 					(unit 1)
 				)
-			)
-		)
-	)
-	(symbol
-		(lib_id "Digikey_LQM2HPN4R7MG0L:LQM2HPN4R7MG0L")
-		(at 55.88 67.31 270)
-		(unit 1)
-		(exclude_from_sim no)
-		(in_bom yes)
-		(on_board yes)
-		(dnp no)
-		(fields_autoplaced yes)
-		(property "Reference" "L2"
-			(at 58.42 66.0399 90)
-			(effects
-				(font
-					(size 1.27 1.27)
-				)
-				(justify left)
-			)
-		)
-		(property "Value" "4.7u"
-			(at 58.42 68.5799 90)
-			(effects
-				(font
-					(size 1.27 1.27)
-				)
-				(justify left)
-			)
-		)
-		(property "Footprint" "LQM2HPN4R7MG0L:INDC2520X100N"
-			(at 55.88 67.31 0)
-			(effects
-				(font
-					(size 1.27 1.27)
-				)
-				(justify bottom)
-				(hide yes)
-			)
-		)
-		(property "Datasheet" ""
-			(at 55.88 67.31 0)
-			(effects
-				(font
-					(size 1.27 1.27)
-				)
-				(hide yes)
-			)
-		)
-		(property "Description" ""
-			(at 55.88 67.31 0)
-			(effects
-				(font
-					(size 1.27 1.27)
-				)
-				(hide yes)
-			)
-		)
-		(pin "2"
-		)
-		(pin "1"
-		)
-		(instances
-			(project ""
-				(path "/4a165a6f-6392-4b15-974f-3ac6900bac37"
-					(reference "L2")
-					(unit 1)
-				)
